File: controller/controller.kicad_sch (KiCad schematic)
At the start: 6 parts, among them J1 Input, J2 Control, J3 Pump, J4 Fan, K1 Auto

Commit message: Update the controller schematics
Parts:
- S1: symbol Switch:SW_DPST -> Switch:SW_SPST
Connections:
- no-connect marks 3 -> 1

Commit message: Controller rev. 2 (single output)
Parts:
- removed J4: Fan, TerminalBlock:TerminalBlock_bornier-2_P5.08mm, symbol Connector:Screw_Terminal_01x02
- J3: value Pump -> Output
Other:
- moved on the sheet: J1, J2, J3, K1, S1
